Commit message: Cylindrical end effector

File: kinova_description/urdf/j2n6s200_standalone.xacro (robot description, xacro)
@@ -24,4 +24,24 @@
   </joint>
   <xacro:property name="robot_root" value="root" />
+          <link name="ee1_link">
+            <visual>
+                <origin xyz="0.0 0.0 0.0" rpy="0.0 0.0 1.5"/>
+                <geometry>
+                    <cylinder radius="0.2" length="0.5"/>
+                </geometry>
+            </visual>
+            <collision>
+                <geometry>
+                    <cylinder radius="0.2" length="0.5"/>
+                </geometry>
+            </collision>
+        </link>
+        <joint name="ee1_joint" type="revolute">
+            <parent link="${prefix}_link_6"/>
+            <child link="ee1_link"/>
+            <axis xyz="0 0 1"/>
+            <limit effort="0" lower="-3.14" upper="3.14" velocity="0.6283185307179586"/>
+            <origin rpy="0 0 0" xyz="0 0 0"/>
+        </joint>
   <xacro:j2n6s200  base_parent="${robot_root}"/>
 </robot>

File: kinova_description/urdf/j2n6s300.xacro (robot description, xacro)
@@ -124,3 +124,155 @@
     <xacro:kinova_3fingers link_hand="${prefix}_link_6" prefix="${prefix}_"/>
     </xacro:macro>
+  <xacro:property name="ee0_length" value="0.2"/>
+  <xacro:property name="ee_radius" value="0.01"/>
+  <xacro:property name="ee0_mass" value="0.1"/>
+  <link name="j2n6s300_ee0_link">
+    <visual>
+    <origin xyz="0 0.0 0" rpy="0.0 0.0 0.0"/>
+      <geometry>
+        <cylinder length="0.2" radius="0.01"/>
+      </geometry>
+      <material name="black"/>
+    </visual>
+    <collision>
+        <origin xyz="0 0.0 0" rpy="0.0 0.0 0.0"/>
+        <geometry>
+            <cylinder length="0.2" radius="0.01"/>
+        </geometry>
+    </collision>
+    <inertial>
+    <!-- Define inertial properties with minimal or placeholder values -->
+    <origin rpy="0 0 0" xyz="0 0 0" />
+    <mass value="0.001" />
+    <inertia ixx="0.001" ixy="0.0" ixz="0.0" iyy="0.001" iyz="0.0" izz="0.001" />
+  </inertial>
+  </link>
+    <joint name="j2n6s300_ee0_joint" type="fixed">
+      <parent link="j2n6s300_link_6"/>
+      <child link="j2n6s300_ee0_link"/>
+      <origin rpy="0 0 0" xyz="0 0 -0.146"/>
+    </joint>
+<!-- End effector link 1-->
+  <link name="j2n6s300_ee1_link">
+    <visual>
+    <origin xyz="0.0 0 0.05" rpy="0.0 0.0 0.0"/>
+      <geometry>
+        <cylinder length="0.1" radius="0.01"/>
+      </geometry>
+      <material name="black"/>
+    </visual>
+    <collision>
+    <origin xyz="0 0 0.05" rpy="0.0 0.0 0.0"/>
+      <geometry>
+        <cylinder length="0.1" radius="0.01"/>
+      </geometry>
+    </collision>
+      <inertial>
+    <!-- Define inertial properties with minimal or placeholder values -->
+    <origin rpy="0 0 0" xyz="0 0 0.05" />
+    <mass value="0.1" />
+    <inertia ixx="8.33e-05" iyy="2.5e-07" izz="2.5e-07" ixy="0" ixz="0" iyz="0"/>
+  </inertial>
+  </link>
+  <joint name="j2n6s300_ee1_joint" type="revolute">
+    <origin rpy="0 1.57 0" xyz="-0.01 0.01 -0.09"/>
+    <parent link="j2n6s300_ee0_link"/>
+    <child link="j2n6s300_ee1_link"/>
+    <axis xyz="0 1 0"/>
+    <limit effort="10" velocity="1" lower="${-2*J_PI}" upper="${2*J_PI}"/>
+      <damping value="100"/>
+      <dynamics damping="1e-02"/>
+  </joint>
+  <transmission name="j2n6s300_ee1_transmission">
+    <type>transmission_interface/SimpleTransmission</type>
+    <joint name="j2n6s300_ee1_joint">
+      <hardwareInterface>hardware_interface/EffortJointInterface</hardwareInterface>
+    </joint>
+    <actuator name="j2n6s300_ee1_actuator">
+      <hardwareInterface>hardware_interface/EffortJointInterface</hardwareInterface>
+      <mechanicalReduction>1</mechanicalReduction>
+    </actuator>
+  </transmission>
+    <!-- <joint name="ee1_joint" type="fixed">
+      <origin rpy="0 1.57 0" xyz="0.0 0 -0.100"/>
+      <parent link="ee0_link"/>
+      <child link="ee1_link"/>
+    </joint> -->
+<!-- End effector link 2-->
+  <link name="j2n6s300_ee2_link">
+    <visual>
+    <origin xyz="0.0 0 0.05" rpy="0.0 0.0 0.0"/>
+      <geometry>
+        <cylinder length="0.1" radius="0.01"/>
+      </geometry>
+      <material name="black"/>
+    </visual>
+    <collision>
+    <origin xyz="0.0 0 0.05" rpy="0.0 0.0 0.0"/>
+      <geometry>
+        <cylinder length="0.1" radius="0.01"/>
+      </geometry>
+    </collision>
+    <inertial>
+    <!-- Define inertial properties with minimal or placeholder values -->
+      <origin rpy="0 0 0" xyz="0.0 0 0.05" />
+      <mass value="0.1" />
+      <inertia ixx="8.33e-05" iyy="2.5e-07" izz="2.5e-07" ixy="0" ixz="0" iyz="0"/>
+    </inertial>
+  </link>
+    <joint name="j2n6s300_ee2_joint" type="revolute">
+      <origin rpy="0 0.0 0" xyz="0.0 0 0.1"/>
+      <parent link="j2n6s300_ee1_link"/>
+      <child link="j2n6s300_ee2_link"/>
+      <axis xyz="1 0 0"/>
+      <limit effort="10" velocity="1" lower="${-2*J_PI}" upper="${2*J_PI}"/>
+      <!-- <damping value="100"/> -->
+      <dynamics damping="1e-02"/>
+    </joint>
+  <transmission name="j2n6s300_ee2_transmission">
+    <type>transmission_interface/SimpleTransmission</type>
+    <joint name="j2n6s300_ee2_joint">
+      <hardwareInterface>hardware_interface/EffortJointInterface</hardwareInterface>
+    </joint>
+    <actuator name="j2n6s300_ee2_actuator">
+      <hardwareInterface>hardware_interface/EffortJointInterface</hardwareInterface>
+      <mechanicalReduction>1</mechanicalReduction>
+    </actuator>
+  </transmission>
+  <link name="j2n6s300_mass_link">
+    <visual>
+    <!--Make a sphere of radius 0.02 mass 1-->
+      <geometry>
+        <sphere radius="0.02"/>
+      </geometry>
+      <material name="black"/>
+    </visual>
+    <collision>
+      <geometry>
+        <sphere radius="0.02"/>
+      </geometry>
+    </collision>
+    <inertial>
+    <!-- Define inertial properties with minimal or placeholder values -->
+      <origin rpy="0 0 0" xyz="0.0 0 0.05" />
+      <mass value="1" />
+      <inertia ixx="6.67e-05" iyy="6.67e-05" izz="6.67e-05" ixy="0" ixz="0" iyz="0"/>
+    </inertial>
+  </link>
+  <joint name="j2n6s300_mass_joint" type="fixed">
+    <origin rpy="0 0 0" xyz="0.0 0 0.1"/>
+    <parent link="j2n6s300_ee2_link"/>
+    <child link="j2n6s300_mass_link"/>
+  </joint>
+    <!-- <joint name="ee2_joint" type="fixed">
+      <origin rpy="0 1.57 0" xyz="0.0 0 0.1"/>
+      <parent link="ee1_link"/>
+      <child link="ee2_link"/>
+    </joint> -->
+  <gazebo reference="j2n6s300_ee1_link">
+    <material>Gazebo/Black</material>
+  </gazebo>
+  <gazebo reference="j2n6s300_mass_link">
+    <material>Gazebo/Black</material>
+  </gazebo>
 </root>

File: kinova_description/urdf/j2n6s300_standalone.xacro (robot description, xacro)
@@ -15,4 +15,5 @@
 	xmlns:xacro="http://www.ros.org/wiki/xacro" name="j2n6s300">
   <xacro:include filename="$(find kinova_description)/urdf/j2n6s300.xacro"/>
+  <xacro:include filename="$(find kinova_description)/urdf/passive_ee.xacro" />
   <xacro:property name="circle1_radius" value="0.85"/>
   <xacro:property name="circle2_radius" value="0.575"/>
@@ -29,164 +30,6 @@
     <origin xyz="0 0 0" rpy="0 0 0" />
   </joint>
-  <!-- Define material properties -->
-  <material name="red">
-    <color rgba="1 0 0 1"/>
-  </material>
-  <material name="green">
-    <color rgba="0 1 0 1"/>
-  </material>
-  <material name="blue">
-    <color rgba="0 0 0 1"/>
-  </material>
-  <material name="black">
-    <color rgba="0 0 0 1"/> <!-- Set the color values (R, G, B, A) -->
-  </material>
-  <!-- Circle 1 -->
-  <link name="circle1_link">
-    <visual>
-      <geometry>
-        <cylinder length="${height}" radius="${circle1_radius}"/>
-      </geometry>
-      <material name="red"/>
-    </visual>
-    <collision>
-      <geometry>
-        <cylinder length="0" radius="0"/>
-      </geometry>
-    </collision>
-    <inertial>
-    <!-- Define inertial properties with minimal or placeholder values -->
-    <origin rpy="0 0 0" xyz="0 0 0" />
-    <mass value="0.001" />
-    <inertia ixx="0.0001" ixy="0.0" ixz="0.0" iyy="0.0001" iyz="0.0" izz="0.0001" />
-  </inertial>
-  </link>
-  <!-- Circle 2 -->
-  <link name="circle2_link">
-    <visual>
-      <geometry>
-        <cylinder length="${height}" radius="${circle2_radius}"/>
-      </geometry>
-      <material name="green"/>
-    </visual>
-      <inertial>
-    <!-- Define inertial properties with minimal or placeholder values -->
-    <origin rpy="0 0 0" xyz="0 0 0" />
-    <mass value="0.001" />
-    <inertia ixx="0.0001" ixy="0.0" ixz="0.0" iyy="0.0001" iyz="0.0" izz="0.0001" />
-  </inertial>
-  </link>
-  <!-- Circle 3 -->
-  <link name="circle3_link">
-    <visual>
-      <geometry>
-        <cylinder length="${height}" radius="${circle3_radius}"/>
-      </geometry>
-      <material name="blue"/>
-    </visual>
-      <inertial>
-    <!-- Define inertial properties with minimal or placeholder values -->
-    <origin rpy="0 0 0" xyz="0 0 0" />
-    <mass value="0.001" />
-    <inertia ixx="0.0001" ixy="0.0" ixz="0.0" iyy="0.0001" iyz="0.0" izz="0.0001" />
-  </inertial>
-  </link>
-  <!-- Line 1-->
-  <link name="line1_link">
-    <visual>
-      <origin rpy="0.0 ${pi/2} ${pi/6}"/>
-      <geometry>
-        <cylinder length="${2*circle1_radius}" radius="${line_width}"/>
-      </geometry>
-      <material name="black"/>
-    </visual>
-      <inertial>
-    <!-- Define inertial properties with minimal or placeholder values -->
-    <origin rpy="0 0 0" xyz="0 0 0" />
-    <mass value="0.001" />
-    <inertia ixx="0.0001" ixy="0.0" ixz="0.0" iyy="0.0001" iyz="0.0" izz="0.0001" />
-  </inertial>
-  </link>
-  <!-- Line 2-->
-  <link name="line2_link">
-    <visual>
-      <origin rpy="0.0 ${pi/2} ${pi/2}"/>
-      <geometry>
-        <cylinder length="${2*circle1_radius}" radius="${line_width}"/>
-      </geometry>
-      <material name="black"/>
-    </visual>
-      <inertial>
-    <!-- Define inertial properties with minimal or placeholder values -->
-    <origin rpy="0 0 0" xyz="0 0 0" />
-    <mass value="0.001" />
-    <inertia ixx="0.0001" ixy="0.0" ixz="0.0" iyy="0.0001" iyz="0.0" izz="0.0001" />
-  </inertial>
-  </link>
-  <!-- Line 3-->
-  <link name="line3_link">
-    <visual>
-    <origin rpy="0.0 ${pi/2} ${-pi/6}"/>
-      <geometry>
-        <cylinder length="${2*circle1_radius}" radius="${line_width}"/>
-      </geometry>
-      <material name="black"/>
-    </visual>
-      <inertial>
-    <!-- Define inertial properties with minimal or placeholder values -->
-    <origin rpy="0 0 0" xyz="0 0 0" />
-    <mass value="0.001" />
-    <inertia ixx="0.0001" ixy="0.0" ixz="0.0" iyy="0.0001" iyz="0.0" izz="0.0001" />
-  </inertial>
-  </link>
-  <joint name="connect_circle_and_world" type="fixed">
-    <child link="circle1_link" />
-    <parent link="root" />
-    <origin xyz="0 0 ${height/2}" rpy="0 0 0" />
-  </joint>
-  <joint name="circle1_joint" type="fixed">
-    <origin xyz="0 0 ${height/2}"/>
-    <parent link="circle1_link"/>
-    <child link="circle2_link"/>
-  </joint>
-  <joint name="circle2_joint" type="fixed">
-    <origin xyz="0 0 ${height/2}"/>
-    <parent link="circle2_link"/>
-    <child link="circle3_link"/>
-  </joint>
-  <joint name="line1_joint" type="fixed">
-    <origin xyz="0 0 ${height/2}"/>
-    <parent link="circle3_link"/>
-    <child link="line1_link"/>
-  </joint>
-  <joint name="line2_joint" type="fixed">
-    <origin xyz="0 0 ${height/2}"/>
-    <parent link="circle3_link"/>
-    <child link="line2_link"/>
-  </joint>
-  <joint name="line3_joint" type="fixed">
-    <origin xyz="0 0 ${height/2}"/>
-    <parent link="circle3_link"/>
-    <child link="line3_link"/>
-  </joint>
-  <gazebo reference="circle1_link">
-    <material>Gazebo/Red</material>
-  </gazebo>
-  <gazebo reference="circle2_link">
-    <material>Gazebo/Blue</material>
-  </gazebo>
-    <gazebo reference="circle3_link">
-    <material>Gazebo/White</material>
-  </gazebo>
-  <gazebo reference="line1_link">
-    <material>Gazebo/Black</material>
-  </gazebo>
-  <gazebo reference="line2_link">
-    <material>Gazebo/Black</material>
-  </gazebo>
-  <gazebo reference="line3_link">
-    <material>Gazebo/Black</material>
-  </gazebo>
   <xacro:property name="robot_root" value="root" />
   <xacro:j2n6s300  base_parent="${robot_root}"/>
+  <xacro:passive_ee base_parent="${robot_root}" />
 </robot>
