Commit message: Working ee

File: kinova_description/urdf/j2n6s300.xacro (robot description, xacro)
@@ -18,4 +18,5 @@
     <!-- Import all Gazebo-customization elements -->
     <xacro:include filename="$(find kinova_description)/urdf/kinova.gazebo" />
+    <xacro:include filename="$(find kinova_description)/urdf/passive_ee.xacro" />
     <xacro:property name="link_base_mesh" value="base" />
     <xacro:property name="link_1_mesh" value="shoulder" />
@@ -124,155 +125,3 @@
     <xacro:kinova_3fingers link_hand="${prefix}_link_6" prefix="${prefix}_"/>
     </xacro:macro>
-  <xacro:property name="ee0_length" value="0.2"/>
-  <xacro:property name="ee_radius" value="0.01"/>
-  <xacro:property name="ee0_mass" value="0.1"/>
-  <link name="j2n6s300_ee0_link">
-    <visual>
-    <origin xyz="0 0.0 0" rpy="0.0 0.0 0.0"/>
-      <geometry>
-        <cylinder length="0.2" radius="0.01"/>
-      </geometry>
-      <material name="black"/>
-    </visual>
-    <collision>
-        <origin xyz="0 0.0 0" rpy="0.0 0.0 0.0"/>
-        <geometry>
-            <cylinder length="0.2" radius="0.01"/>
-        </geometry>
-    </collision>
-    <inertial>
-    <!-- Define inertial properties with minimal or placeholder values -->
-    <origin rpy="0 0 0" xyz="0 0 0" />
-    <mass value="0.001" />
-    <inertia ixx="0.001" ixy="0.0" ixz="0.0" iyy="0.001" iyz="0.0" izz="0.001" />
-  </inertial>
-  </link>
-    <joint name="j2n6s300_ee0_joint" type="fixed">
-      <parent link="j2n6s300_link_6"/>
-      <child link="j2n6s300_ee0_link"/>
-      <origin rpy="0 0 0" xyz="0 0 -0.146"/>
-    </joint>
-<!-- End effector link 1-->
-  <link name="j2n6s300_ee1_link">
-    <visual>
-    <origin xyz="0.0 0 0.05" rpy="0.0 0.0 0.0"/>
-      <geometry>
-        <cylinder length="0.1" radius="0.01"/>
-      </geometry>
-      <material name="black"/>
-    </visual>
-    <collision>
-    <origin xyz="0 0 0.05" rpy="0.0 0.0 0.0"/>
-      <geometry>
-        <cylinder length="0.1" radius="0.01"/>
-      </geometry>
-    </collision>
-      <inertial>
-    <!-- Define inertial properties with minimal or placeholder values -->
-    <origin rpy="0 0 0" xyz="0 0 0.05" />
-    <mass value="0.1" />
-    <inertia ixx="8.33e-05" iyy="2.5e-07" izz="2.5e-07" ixy="0" ixz="0" iyz="0"/>
-  </inertial>
-  </link>
-  <joint name="j2n6s300_ee1_joint" type="revolute">
-    <origin rpy="0 1.57 0" xyz="-0.01 0.01 -0.09"/>
-    <parent link="j2n6s300_ee0_link"/>
-    <child link="j2n6s300_ee1_link"/>
-    <axis xyz="0 1 0"/>
-    <limit effort="10" velocity="1" lower="${-2*J_PI}" upper="${2*J_PI}"/>
-      <damping value="100"/>
-      <dynamics damping="1e-02"/>
-  </joint>
-  <transmission name="j2n6s300_ee1_transmission">
-    <type>transmission_interface/SimpleTransmission</type>
-    <joint name="j2n6s300_ee1_joint">
-      <hardwareInterface>hardware_interface/EffortJointInterface</hardwareInterface>
-    </joint>
-    <actuator name="j2n6s300_ee1_actuator">
-      <hardwareInterface>hardware_interface/EffortJointInterface</hardwareInterface>
-      <mechanicalReduction>1</mechanicalReduction>
-    </actuator>
-  </transmission>
-    <!-- <joint name="ee1_joint" type="fixed">
-      <origin rpy="0 1.57 0" xyz="0.0 0 -0.100"/>
-      <parent link="ee0_link"/>
-      <child link="ee1_link"/>
-    </joint> -->
-<!-- End effector link 2-->
-  <link name="j2n6s300_ee2_link">
-    <visual>
-    <origin xyz="0.0 0 0.05" rpy="0.0 0.0 0.0"/>
-      <geometry>
-        <cylinder length="0.1" radius="0.01"/>
-      </geometry>
-      <material name="black"/>
-    </visual>
-    <collision>
-    <origin xyz="0.0 0 0.05" rpy="0.0 0.0 0.0"/>
-      <geometry>
-        <cylinder length="0.1" radius="0.01"/>
-      </geometry>
-    </collision>
-    <inertial>
-    <!-- Define inertial properties with minimal or placeholder values -->
-      <origin rpy="0 0 0" xyz="0.0 0 0.05" />
-      <mass value="0.1" />
-      <inertia ixx="8.33e-05" iyy="2.5e-07" izz="2.5e-07" ixy="0" ixz="0" iyz="0"/>
-    </inertial>
-  </link>
-    <joint name="j2n6s300_ee2_joint" type="revolute">
-      <origin rpy="0 0.0 0" xyz="0.0 0 0.1"/>
-      <parent link="j2n6s300_ee1_link"/>
-      <child link="j2n6s300_ee2_link"/>
-      <axis xyz="1 0 0"/>
-      <limit effort="10" velocity="1" lower="${-2*J_PI}" upper="${2*J_PI}"/>
-      <!-- <damping value="100"/> -->
-      <dynamics damping="1e-02"/>
-    </joint>
-  <transmission name="j2n6s300_ee2_transmission">
-    <type>transmission_interface/SimpleTransmission</type>
-    <joint name="j2n6s300_ee2_joint">
-      <hardwareInterface>hardware_interface/EffortJointInterface</hardwareInterface>
-    </joint>
-    <actuator name="j2n6s300_ee2_actuator">
-      <hardwareInterface>hardware_interface/EffortJointInterface</hardwareInterface>
-      <mechanicalReduction>1</mechanicalReduction>
-    </actuator>
-  </transmission>
-  <link name="j2n6s300_mass_link">
-    <visual>
-    <!--Make a sphere of radius 0.02 mass 1-->
-      <geometry>
-        <sphere radius="0.02"/>
-      </geometry>
-      <material name="black"/>
-    </visual>
-    <collision>
-      <geometry>
-        <sphere radius="0.02"/>
-      </geometry>
-    </collision>
-    <inertial>
-    <!-- Define inertial properties with minimal or placeholder values -->
-      <origin rpy="0 0 0" xyz="0.0 0 0.05" />
-      <mass value="1" />
-      <inertia ixx="6.67e-05" iyy="6.67e-05" izz="6.67e-05" ixy="0" ixz="0" iyz="0"/>
-    </inertial>
-  </link>
-  <joint name="j2n6s300_mass_joint" type="fixed">
-    <origin rpy="0 0 0" xyz="0.0 0 0.1"/>
-    <parent link="j2n6s300_ee2_link"/>
-    <child link="j2n6s300_mass_link"/>
-  </joint>
-    <!-- <joint name="ee2_joint" type="fixed">
-      <origin rpy="0 1.57 0" xyz="0.0 0 0.1"/>
-      <parent link="ee1_link"/>
-      <child link="ee2_link"/>
-    </joint> -->
-  <gazebo reference="j2n6s300_ee1_link">
-    <material>Gazebo/Black</material>
-  </gazebo>
-  <gazebo reference="j2n6s300_mass_link">
-    <material>Gazebo/Black</material>
-  </gazebo>
 </root>

File: kinova_description/urdf/j2n6s300_standalone.xacro (robot description, xacro)
@@ -15,5 +15,4 @@
 	xmlns:xacro="http://www.ros.org/wiki/xacro" name="j2n6s300">
   <xacro:include filename="$(find kinova_description)/urdf/j2n6s300.xacro"/>
-  <xacro:include filename="$(find kinova_description)/urdf/passive_ee.xacro" />
   <xacro:property name="circle1_radius" value="0.85"/>
   <xacro:property name="circle2_radius" value="0.575"/>
@@ -32,4 +31,4 @@
   <xacro:property name="robot_root" value="root" />
   <xacro:j2n6s300  base_parent="${robot_root}"/>
-  <xacro:passive_ee base_parent="${robot_root}" />
+  <xacro:passive_ee base_parent="j2n6s300_link_6"/>
 </robot>

File: kinova_description/urdf/passive_ee.xacro (robot description, xacro)
@@ -1,6 +1,7 @@
 <?xml version="1.0"?>
 <robot xmlns:xacro="http://www.ros.org/wiki/xacro" name="passive_ees">
+    <xacro:property name="pi" value="3.14159265359"/>
   <!-- Define the macro to generate a cuboid link -->
-  <xacro:macro name="passive_ee_link" params="parent name length width height mass color xyz rpy joint_type joint_revolute_axis">
+  <xacro:macro name="passive_ee_link" params="parent name length width height mass color xyz rpy joint_xyz joint_rpy joint_type joint_revolute_axis">
     <link name="${name}_link">
       <visual>
@@ -23,18 +24,20 @@
         <origin xyz="${xyz}" rpy="${rpy}" />
         <inertia
-          ixx="${0.0833 * mass * (width * width + height * height)}"
+          ixx="${(1.0/12.0) * mass * (width * width + height * height)}"
           ixy="0.0"
           ixz="0.0"
-          iyy="${0.0833 * mass * (length * length + height * height)}"
+          iyy="${(1.0/12.0) * mass * (length * length + height * height)}"
           iyz="0.0"
-          izz="${0.0833 * mass * (length * length + width * width)}" />
+          izz="${(1.0/12.0) * mass * (length * length + width * width)}" />
       </inertial>
     </link>
-    <joint name="${name}_joint" type="fixed">
+    <joint name="${name}_joint" type="${joint_type}">
         <parent link="${parent}" />
         <child link="${name}_link" />
-        <origin xyz="${xyz}" rpy="${rpy}" />
+        <origin xyz="${joint_xyz}" rpy="${joint_rpy}" />
         <xacro:if value="${joint_type == 'revolute'}">
             <axis xyz="${joint_revolute_axis}" />
+            <limit effort="100" velocity="5" lower="${-2*pi}" upper="${2*pi}"/>
+            <dynamics damping="1e-02"/>
         </xacro:if>
     </joint>
@@ -43,8 +46,8 @@
         <transmission name="${name}_joint_transmission">
             <type>transmission_interface/SimpleTransmission</type>
-            <joint name="{name}_joint">
+            <joint name="${name}_joint">
                 <hardwareInterface>hardware_interface/EffortJointInterface</hardwareInterface>
             </joint>
-            <actuator name="{name}_joint_actuator">
+            <actuator name="${name}_joint_actuator">
                 <hardwareInterface>hardware_interface/EffortJointInterface</hardwareInterface>
                 <mechanicalReduction>1</mechanicalReduction>
@@ -53,15 +56,64 @@
     </xacro:if>
   </xacro:macro>
+<!-- Define the macro to generate a cylinder link -->
+  <xacro:macro name="passive_ee_mass" params="parent name radius height mass color xyz joint_xyz">
+    <link name="${name}_link">
+      <visual>
+        <geometry>
+          <cylinder radius="${radius}" length="${height}" />
+        </geometry>
+        <material name="${name}_material">
+          <color rgba="${color}" />
+        </material>
+      </visual>
+      <collision>
+        <geometry>
+          <cylinder radius="${radius}" length="${height}" />
+        </geometry>
+      </collision>
+      <inertial>
+        <mass value="${mass}" />
+        <origin xyz="${xyz}" rpy="0 0 0" />
+        <inertia
+          ixx="${(1.0/12.0) * mass * (3 * radius * radius + height * height)}"
+          ixy="0.0"
+          ixz="0.0"
+          iyy="${(1.0/12.0) * mass * (3 * radius * radius + height * height)}"
+          iyz="0.0"
+          izz="${(1.0/2.0) * mass * radius * radius}" />
+      </inertial>
+    </link>
+    <joint name="fixed_joint_${name}" type="fixed">
+      <parent link="${parent}" />
+      <child link="${name}_link" />
+      <origin xyz="${joint_xyz}" rpy="0 0 0" />
+    </joint>
+  </xacro:macro>
   <!-- Define the properties for each cuboid link -->
+  <!-- Define passive_ee_0-->
+    <xacro:property name="passive_ee_0_name" value="passive_ee_0" />
+    <xacro:property name="passive_ee_0_length" value="0.02" />
+    <xacro:property name="passive_ee_0_width" value="0.02" />
+    <xacro:property name="passive_ee_0_height" value="0.2" />
+    <xacro:property name="passive_ee_0_mass" value="0.2" />
+    <xacro:property name="passive_ee_0_color" value="0.0 0.0 1.0 1.0" />
+    <xacro:property name="passive_ee_0_xyz" value="0.0 0.0 ${-passive_ee_0_height/2}" />
+    <xacro:property name="passive_ee_0_rpy" value="0.0 0.0 0.0" />
+    <xacro:property name="passive_ee_0_joint_xyz" value="0.0 0.0 -0.12" /> <!-- 0.12 is the distance between link 6 frame and top of palm -->
+    <xacro:property name="passive_ee_0_joint_rpy" value="0.0 0.0 0.0" />
+    <xacro:property name="passive_ee_0_joint_type" value="fixed" />
+    <xacro:property name="passive_ee_0_joint_revolute_axis" value="0.0 0.0 0.0" />
   <xacro:property name="passive_ee_1_name" value="passive_ee_1" />
   <xacro:property name="passive_ee_1_length" value="0.02" />
   <xacro:property name="passive_ee_1_width" value="0.02" />
-  <xacro:property name="passive_ee_1_height" value="0.1" />
-  <xacro:property name="passive_ee_1_mass" value="1.0" />
+  <xacro:property name="passive_ee_1_height" value="0.10" />
+  <xacro:property name="passive_ee_1_mass" value="0.10" />
   <xacro:property name="passive_ee_1_color" value="0.0 1.0 0.0 1.0" />
-  <xacro:property name="passive_ee_1_xyz" value="0.0 0.0 0.0" />
+  <xacro:property name="passive_ee_1_xyz" value="0.0 0.0 ${-passive_ee_1_height/2}" />
     <xacro:property name="passive_ee_1_rpy" value="0.0 0.0 0.0" />
-    <xacro:property name="passive_ee_1_joint_type" value="fixed" />
-    <xacro:property name="passive_ee_1_joint_revolute_axis" value="0.0 0.0 0.0" />
+    <xacro:property name="passive_ee_1_joint_xyz" value="${passive_ee_1_width} 0.0 ${-passive_ee_0_height+passive_ee_1_width/2}" />
+    <xacro:property name="passive_ee_1_joint_rpy" value="0.0 0.0 0.0" />
+    <xacro:property name="passive_ee_1_joint_type" value="revolute" />
+    <xacro:property name="passive_ee_1_joint_revolute_axis" value="1.0 0.0 0.0" />
   <!-- Gazebo material reference for passive_ee_1 -->
   <xacro:property name="passive_ee_1_gazebo_material" value="Gazebo/Green" />
@@ -69,11 +121,20 @@
   <xacro:property name="passive_ee_2_length" value="0.02" />
   <xacro:property name="passive_ee_2_width" value="0.02" />
-  <xacro:property name="passive_ee_2_height" value="0.1" />
-  <xacro:property name="passive_ee_2_mass" value="0.5" />
+  <xacro:property name="passive_ee_2_height" value="0.10" />
+  <xacro:property name="passive_ee_2_mass" value="0.10" />
   <xacro:property name="passive_ee_2_color" value="1.0 0.0 0.0 1.0" />
-  <xacro:property name="passive_ee_2_xyz" value="1.0 0.0 0.0" />
+  <xacro:property name="passive_ee_2_xyz" value="0.0 0.0 ${-passive_ee_2_height/2}" />
     <xacro:property name="passive_ee_2_rpy" value="0.0 0.0 0.0" />
-    <xacro:property name="passive_ee_2_joint_type" value="fixed" />
-    <xacro:property name="passive_ee_2_joint_revolute_axis" value="0.0 0.0 0.0" />
+    <xacro:property name="passive_ee_2_joint_xyz" value="0.0 ${passive_ee_2_width} ${-passive_ee_1_height+passive_ee_2_width/2}" />
+    <xacro:property name="passive_ee_2_joint_rpy" value="0.0 0.0 0.0" />
+    <xacro:property name="passive_ee_2_joint_type" value="revolute" />
+    <xacro:property name="passive_ee_2_joint_revolute_axis" value="0.0 1.0 0.0" />
+    <xacro:property name="passive_ee_mass_name" value="passive_ee_mass" />
+    <xacro:property name="passive_ee_mass_radius" value = "0.03" />
+    <xacro:property name="passive_ee_mass_height" value = "0.03" />
+    <xacro:property name="passive_ee_mass_mass" value = "1.0" />
+    <xacro:property name="passive_ee_mass_color" value = "0.0 0.0 0.0 1.0" />
+    <xacro:property name="passive_ee_mass_xyz" value="0.0 0.0 0.0" />
+    <xacro:property name="passive_ee_mass_joint_xyz" value="0.0 0.0 ${-passive_ee_2_height-passive_ee_mass_height/2}" />
   <!-- Gazebo material reference for passive_ee_2 -->
   <xacro:property name="passive_ee_2_gazebo_material" value="Gazebo/Red" />
@@ -82,4 +143,19 @@
     <xacro:passive_ee_link
         parent="${base_parent}"
+        name="${passive_ee_0_name}"
+        length="${passive_ee_0_length}"
+        width="${passive_ee_0_width}"
+        height="${passive_ee_0_height}"
+        mass="${passive_ee_0_mass}"
+        color="${passive_ee_0_color}"
+        xyz="${passive_ee_0_xyz}"
+        rpy="${passive_ee_0_rpy}"
+        joint_xyz="${passive_ee_0_joint_xyz}"
+        joint_rpy="${passive_ee_0_joint_rpy}"
+        joint_type="${passive_ee_0_joint_type}"
+        joint_revolute_axis="${passive_ee_0_joint_revolute_axis}"
+    />
+    <xacro:passive_ee_link
+        parent="${passive_ee_0_name}_link"
         name="${passive_ee_1_name}"
         length="${passive_ee_1_length}"
@@ -90,4 +166,6 @@
         xyz="${passive_ee_1_xyz}"
         rpy="${passive_ee_1_rpy}"
+        joint_xyz="${passive_ee_1_joint_xyz}"
+        joint_rpy="${passive_ee_1_joint_rpy}"
         joint_type="${passive_ee_1_joint_type}"
         joint_revolute_axis="${passive_ee_1_joint_revolute_axis}"
@@ -103,6 +181,18 @@
         xyz="${passive_ee_2_xyz}"
         rpy="${passive_ee_2_rpy}"
+        joint_xyz="${passive_ee_2_joint_xyz}"
+        joint_rpy="${passive_ee_2_joint_rpy}"
         joint_type="${passive_ee_2_joint_type}"
         joint_revolute_axis="${passive_ee_2_joint_revolute_axis}"
+    />
+    <xacro:passive_ee_mass
+        parent="${passive_ee_2_name}_link"
+        name="${passive_ee_mass_name}"
+        radius="${passive_ee_mass_radius}"
+        height="${passive_ee_mass_height}"
+        mass="${passive_ee_mass_mass}"
+        color="${passive_ee_mass_color}"
+        xyz="${passive_ee_mass_xyz}"
+        joint_xyz="${passive_ee_mass_joint_xyz}"
     />
     </xacro:macro>
@@ -116,3 +206,23 @@
     </material>
   </gazebo>
+  <gazebo reference="passive_ee_1_link">
+    <gravity>true</gravity>
+    <sensor name="imu_sensor" type="imu">
+      <always_on>true</always_on>
+      <update_rate>100</update_rate>
+      <visualize>true</visualize>
+      <topic>/passive_ee_1_imu</topic>
+      <plugin filename="libgazebo_ros_imu_sensor.so" name="imu_plugin">
+        <topicName>/passive_ee_1_imu</topicName>
+        <bodyName>passive_ee1_link</bodyName>
+        <updateRateHZ>10.0</updateRateHZ>
+        <gaussianNoise>0.0</gaussianNoise>
+        <xyzOffset>0 0 ${-passive_ee_1_height/2}</xyzOffset>
+        <rpyOffset>0 0 0</rpyOffset>
+        <frameName>passive_ee_1_link</frameName>
+        <initialOrientationAsReference>false</initialOrientationAsReference>
+      </plugin>
+      <pose>0 0 0 0 0 0</pose>
+    </sensor>
+  </gazebo>
 </robot>
