Commit message: Added circle world

File: kinova_description/urdf/j2n6s300_standalone.xacro (robot description, xacro)
@@ -15,7 +15,13 @@
 	xmlns:xacro="http://www.ros.org/wiki/xacro" name="j2n6s300">
   <xacro:include filename="$(find kinova_description)/urdf/j2n6s300.xacro"/>
-  <link name="root"/>
+  <xacro:property name="circle1_radius" value="0.85"/>
+  <xacro:property name="circle2_radius" value="0.575"/>
+  <xacro:property name="circle3_radius" value="0.3"/>
+  <xacro:property name="height" value="0.001"/>
+  <xacro:property name="line_width" value="0.01"/>
+  <xacro:property name="pi" value="3.14159265359"/>
   <!-- for gazebo -->
   <link name="world"/>
+  <link name="root"/>
   <joint name="connect_root_and_world" type="fixed">
     <child link="root" />
@@ -23,4 +29,163 @@
     <origin xyz="0 0 0" rpy="0 0 0" />
   </joint>
+  <!-- Define material properties -->
+  <material name="red">
+    <color rgba="1 0 0 1"/>
+  </material>
+  <material name="green">
+    <color rgba="0 1 0 1"/>
+  </material>
+  <material name="blue">
+    <color rgba="0 0 0 1"/>
+  </material>
+  <material name="black">
+    <color rgba="0 0 0 1"/> <!-- Set the color values (R, G, B, A) -->
+  </material>
+  <!-- Circle 1 -->
+  <link name="circle1_link">
+    <visual>
+      <geometry>
+        <cylinder length="${height}" radius="${circle1_radius}"/>
+      </geometry>
+      <material name="red"/>
+    </visual>
+    <collision>
+      <geometry>
+        <cylinder length="0" radius="0"/>
+      </geometry>
+    </collision>
+    <inertial>
+    <!-- Define inertial properties with minimal or placeholder values -->
+    <origin rpy="0 0 0" xyz="0 0 0" />
+    <mass value="0.001" />
+    <inertia ixx="0.0001" ixy="0.0" ixz="0.0" iyy="0.0001" iyz="0.0" izz="0.0001" />
+  </inertial>
+  </link>
+  <!-- Circle 2 -->
+  <link name="circle2_link">
+    <visual>
+      <geometry>
+        <cylinder length="${height}" radius="${circle2_radius}"/>
+      </geometry>
+      <material name="green"/>
+    </visual>
+      <inertial>
+    <!-- Define inertial properties with minimal or placeholder values -->
+    <origin rpy="0 0 0" xyz="0 0 0" />
+    <mass value="0.001" />
+    <inertia ixx="0.0001" ixy="0.0" ixz="0.0" iyy="0.0001" iyz="0.0" izz="0.0001" />
+  </inertial>
+  </link>
+  <!-- Circle 3 -->
+  <link name="circle3_link">
+    <visual>
+      <geometry>
+        <cylinder length="${height}" radius="${circle3_radius}"/>
+      </geometry>
+      <material name="blue"/>
+    </visual>
+      <inertial>
+    <!-- Define inertial properties with minimal or placeholder values -->
+    <origin rpy="0 0 0" xyz="0 0 0" />
+    <mass value="0.001" />
+    <inertia ixx="0.0001" ixy="0.0" ixz="0.0" iyy="0.0001" iyz="0.0" izz="0.0001" />
+  </inertial>
+  </link>
+  <!-- Line 1-->
+  <link name="line1_link">
+    <visual>
+      <origin rpy="0.0 ${pi/2} 0.0"/>
+      <geometry>
+        <cylinder length="${2*circle1_radius}" radius="${line_width}"/>
+      </geometry>
+      <material name="black"/>
+    </visual>
+      <inertial>
+    <!-- Define inertial properties with minimal or placeholder values -->
+    <origin rpy="0 0 0" xyz="0 0 0" />
+    <mass value="0.001" />
+    <inertia ixx="0.0001" ixy="0.0" ixz="0.0" iyy="0.0001" iyz="0.0" izz="0.0001" />
+  </inertial>
+  </link>
+  <!-- Line 2-->
+  <link name="line2_link">
+    <visual>
+      <origin rpy="0.0 ${pi/2} ${pi/3}"/>
+      <geometry>
+        <cylinder length="${2*circle1_radius}" radius="${line_width}"/>
+      </geometry>
+      <material name="black"/>
+    </visual>
+      <inertial>
+    <!-- Define inertial properties with minimal or placeholder values -->
+    <origin rpy="0 0 0" xyz="0 0 0" />
+    <mass value="0.001" />
+    <inertia ixx="0.0001" ixy="0.0" ixz="0.0" iyy="0.0001" iyz="0.0" izz="0.0001" />
+  </inertial>
+  </link>
+  <!-- Line 3-->
+  <link name="line3_link">
+    <visual>
+    <origin rpy="0.0 ${pi/2} ${-pi/3}"/>
+      <geometry>
+        <cylinder length="${2*circle1_radius}" radius="${line_width}"/>
+      </geometry>
+      <material name="black"/>
+    </visual>
+      <inertial>
+    <!-- Define inertial properties with minimal or placeholder values -->
+    <origin rpy="0 0 0" xyz="0 0 0" />
+    <mass value="0.001" />
+    <inertia ixx="0.0001" ixy="0.0" ixz="0.0" iyy="0.0001" iyz="0.0" izz="0.0001" />
+  </inertial>
+  </link>
+  <joint name="connect_circle_and_world" type="fixed">
+    <child link="circle1_link" />
+    <parent link="root" />
+    <origin xyz="0 0 ${height/2}" rpy="0 0 0" />
+  </joint>
+  <joint name="circle1_joint" type="fixed">
+    <origin xyz="0 0 ${height/2}"/>
+    <parent link="circle1_link"/>
+    <child link="circle2_link"/>
+  </joint>
+  <joint name="circle2_joint" type="fixed">
+    <origin xyz="0 0 ${height/2}"/>
+    <parent link="circle2_link"/>
+    <child link="circle3_link"/>
+  </joint>
+  <joint name="line1_joint" type="fixed">
+    <origin xyz="0 0 ${height/2}"/>
+    <parent link="circle3_link"/>
+    <child link="line1_link"/>
+  </joint>
+  <joint name="line2_joint" type="fixed">
+    <origin xyz="0 0 ${height/2}"/>
+    <parent link="circle3_link"/>
+    <child link="line2_link"/>
+  </joint>
+  <joint name="line3_joint" type="fixed">
+    <origin xyz="0 0 ${height/2}"/>
+    <parent link="circle3_link"/>
+    <child link="line3_link"/>
+  </joint>
+  <gazebo reference="circle1_link">
+    <material>Gazebo/Red</material>
+  </gazebo>
+  <gazebo reference="circle2_link">
+    <material>Gazebo/Blue</material>
+  </gazebo>
+    <gazebo reference="circle3_link">
+    <material>Gazebo/White</material>
+  </gazebo>
+  <gazebo reference="line1_link">
+    <material>Gazebo/Black</material>
+  </gazebo>
+  <gazebo reference="line2_link">
+    <material>Gazebo/Black</material>
+  </gazebo>
+  <gazebo reference="line3_link">
+    <material>Gazebo/Black</material>
+  </gazebo>
   <xacro:property name="robot_root" value="root" />
   <xacro:j2n6s300  base_parent="${robot_root}"/>

Commit message: Fixed circle lines

File: kinova_description/urdf/j2n6s300_standalone.xacro (robot description, xacro)
@@ -95,5 +95,5 @@
   <link name="line1_link">
     <visual>
-      <origin rpy="0.0 ${pi/2} 0.0"/>
+      <origin rpy="0.0 ${pi/2} ${pi/6}"/>
       <geometry>
         <cylinder length="${2*circle1_radius}" radius="${line_width}"/>
@@ -111,5 +111,5 @@
   <link name="line2_link">
     <visual>
-      <origin rpy="0.0 ${pi/2} ${pi/3}"/>
+      <origin rpy="0.0 ${pi/2} ${pi/2}"/>
       <geometry>
         <cylinder length="${2*circle1_radius}" radius="${line_width}"/>
@@ -127,5 +127,5 @@
   <link name="line3_link">
     <visual>
-    <origin rpy="0.0 ${pi/2} ${-pi/3}"/>
+    <origin rpy="0.0 ${pi/2} ${-pi/6}"/>
       <geometry>
         <cylinder length="${2*circle1_radius}" radius="${line_width}"/>

Commit message: Updated circle radii

File: kinova_description/urdf/j2n6s300_standalone.xacro (robot description, xacro)
@@ -15,7 +15,7 @@
 	xmlns:xacro="http://www.ros.org/wiki/xacro" name="j2n6s300">
   <xacro:include filename="$(find kinova_description)/urdf/j2n6s300.xacro"/>
-  <xacro:property name="circle1_radius" value="0.85"/>
-  <xacro:property name="circle2_radius" value="0.575"/>
-  <xacro:property name="circle3_radius" value="0.3"/>
+  <xacro:property name="circle1_radius" value="0.75"/>
+  <xacro:property name="circle2_radius" value="0.475"/>
+  <xacro:property name="circle3_radius" value="0.2"/>
   <xacro:property name="height" value="0.001"/>
   <xacro:property name="line_width" value="0.01"/>

File: kinova_description/urdf/kinova_common.xacro (robot description, xacro)
@@ -85,5 +85,5 @@
         </xacro:if>
         <origin xyz="${joint_origin_xyz}" rpy="${joint_origin_rpy}"/>
-        <dynamics damping="0.0" friction="0.0"/>
+        <dynamics damping="0.1" friction="0.0"/>
      </joint>
    <xacro:unless value="${fixed}">

Commit message: Added new plugins for joint states and control

File: kinova_description/urdf/j2n6s300_standalone.xacro (robot description, xacro)
@@ -15,10 +15,28 @@
 	xmlns:xacro="http://www.ros.org/wiki/xacro" name="j2n6s300">
   <xacro:include filename="$(find kinova_description)/urdf/j2n6s300.xacro"/>
-  <xacro:property name="circle1_radius" value="0.85"/>
-  <xacro:property name="circle2_radius" value="0.575"/>
-  <xacro:property name="circle3_radius" value="0.3"/>
-  <xacro:property name="height" value="0.001"/>
-  <xacro:property name="line_width" value="0.01"/>
-  <xacro:property name="pi" value="3.14159265359"/>
+  <!-- Define the link -->
+  <link name="base_link">
+    <visual>
+      <geometry>
+        <box size="0.1 0.1 0.5"/>
+      </geometry>
+    </visual>
+    <collision>
+      <geometry>
+        <box size="0.1 0.1 0.5"/>
+      </geometry>
+    </collision>
+    <inertial>
+      <mass value="1"/>
+      <origin rpy="0 0 0" xyz="0 0 0"/>
+      <inertia ixx="0.00416667" ixy="0" ixz="0" iyy="0.00416667" iyz="0" izz="0.00416667"/>
+    </inertial>
+  </link>
+  <!-- Define the joint -->
+  <joint name="fixed_joint" type="fixed">
+    <parent link="world"/>
+    <child link="base_link"/>
+    <origin rpy="0 0 0" xyz="0 0 0.25"/>
+  </joint>
   <!-- for gazebo -->
   <link name="world"/>
@@ -26,9 +44,15 @@
   <joint name="connect_root_and_world" type="fixed">
     <child link="root" />
-    <parent link="world" />
-    <origin xyz="0 0 0" rpy="0 0 0" />
+    <parent link="base_link" />
+    <origin xyz="0 0 0.25" rpy="0 0 0" />
   </joint>
   <xacro:property name="robot_root" value="root" />
   <xacro:j2n6s300  base_parent="${robot_root}"/>
   <xacro:passive_ee base_parent="j2n6s300_link_6"/>
+    <!-- Add the plugin to the robot -->
+  <gazebo>
+    <plugin name="fast_joints_plugin" filename="libfast_joints_plugin.so">
+      <!-- Plugin parameters, if any -->
+    </plugin>
+  </gazebo>
 </robot>

File: kinova_description/urdf/passive_ee.xacro (robot description, xacro)
@@ -21,5 +21,5 @@
       </collision>
       <inertial>
-        <mass value="${mass}" />
+        <mass value="5e-04" />
         <origin xyz="${xyz}" rpy="${rpy}" />
         <inertia
@@ -39,5 +39,5 @@
             <axis xyz="${joint_revolute_axis}" />
             <limit effort="100" velocity="5" lower="${-2*pi}" upper="${2*pi}"/>
-            <dynamics damping="0.4"/>
+            <dynamics damping="0.004"/>
         </xacro:if>
     </joint>
@@ -95,6 +95,6 @@
     <xacro:property name="passive_ee_0_length" value="0.02" />
     <xacro:property name="passive_ee_0_width" value="0.02" />
-    <xacro:property name="passive_ee_0_height" value="0.1" />
-    <xacro:property name="passive_ee_0_mass" value="0.1" />
+    <xacro:property name="passive_ee_0_height" value="0.15" />
+    <xacro:property name="passive_ee_0_mass" value="1e-03" />
     <xacro:property name="passive_ee_0_color" value="0.0 0.0 1.0 1.0" />
     <xacro:property name="passive_ee_0_xyz" value="0.0 0.0 ${-passive_ee_0_height/2}" />
@@ -108,5 +108,5 @@
   <xacro:property name="passive_ee_1_width" value="0.02" />
   <xacro:property name="passive_ee_1_height" value="0.1" />
-  <xacro:property name="passive_ee_1_mass" value="0.1" />
+  <xacro:property name="passive_ee_1_mass" value="1e-03" />
   <xacro:property name="passive_ee_1_color" value="0.0 1.0 0.0 1.0" />
   <xacro:property name="passive_ee_1_xyz" value="0.0 0.0 ${-passive_ee_1_height/2}" />
@@ -123,5 +123,5 @@
   <xacro:property name="middle_link_1_width" value="0.005" />
   <xacro:property name="middle_link_1_height" value="0.04" />
-  <xacro:property name="middle_link_1_mass" value="0.001" />
+  <xacro:property name="middle_link_1_mass" value="1e-03" />
   <xacro:property name="middle_link_1_color" value="0.0 0.0 0.0 1.0" />
   <xacro:property name="middle_link_1_xyz" value="0.0 0.0 ${-middle_link_1_height/2}" />
@@ -136,5 +136,5 @@
   <xacro:property name="middle_link_2_width" value="0.005" />
   <xacro:property name="middle_link_2_height" value="0.04" />
-  <xacro:property name="middle_link_2_mass" value="0.001" />
+  <xacro:property name="middle_link_2_mass" value="1e-03" />
   <xacro:property name="middle_link_2_color" value="0.0 0.0 0.0 1.0" />
   <xacro:property name="middle_link_2_xyz" value="0.0 0.0 ${-middle_link_2_height/2}" />
@@ -148,5 +148,5 @@
   <xacro:property name="passive_ee_2_width" value="0.02" />
   <xacro:property name="passive_ee_2_height" value="0.2" />
-  <xacro:property name="passive_ee_2_mass" value="0.2" />
+  <xacro:property name="passive_ee_2_mass" value="1e-03" />
   <xacro:property name="passive_ee_2_color" value="1.0 0.0 0.0 1.0" />
   <xacro:property name="passive_ee_2_xyz" value="0.0 0.0 ${-passive_ee_2_height/2}" />

Commit message: Change joystick readings

File: kinova_description/urdf/j2n6s300_standalone.xacro (robot description, xacro)
@@ -15,7 +15,7 @@
 	xmlns:xacro="http://www.ros.org/wiki/xacro" name="j2n6s300">
   <xacro:include filename="$(find kinova_description)/urdf/j2n6s300.xacro"/>
-  <xacro:property name="circle1_radius" value="0.75"/>
-  <xacro:property name="circle2_radius" value="0.475"/>
-  <xacro:property name="circle3_radius" value="0.2"/>
+  <xacro:property name="circle1_radius" value="0.85"/>
+  <xacro:property name="circle2_radius" value="0.575"/>
+  <xacro:property name="circle3_radius" value="0.3"/>
   <xacro:property name="height" value="0.001"/>
   <xacro:property name="line_width" value="0.01"/>
